File: CB350/CB350.kicad_pcb (KiCad board)
At the start: 4 copper layers, 25 x 50 mm, 56 parts, among them J1 V_In, J10 GND, J2 GND, J3 5V, J4 GND, J5 S, J6 S, J7 V+, J8 G, J9 V_Out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

Commit message: Overhaul
Parts:
- moved REF** 25.4 mm to (108.7, 64.2)
- moved REF** 18.4 mm to (116.1, 57.2)
- moved REF** 18.2 mm to (116.0, 64.1)
- moved G*** 7.52 mm to (116.0, 73.3)
Routing:
- net GND: vias 23 -> 25
Other:
- board text added: "github.com/Synthron/SY317/CB350"
