File: CB350/CB350.kicad_sch (KiCad schematic)
At the start: 46 parts, among them J101 V_In, J102 GND, J103 V+, J104 G, J105 S, J106 S, U101 SIC471ED-T1-GE3

Commit message: Update CB350 files, cleanup repo
Parts:
- removed C101: 47µ R07, symbol Device:C_Polarized
- added C1: 47µ, Capacitor_SMD:C_1210_3225Metric, symbol Device:C
- added J10: GND, TestPoint:TestPoint_THTPad_4.0x4.0mm_Drill2.0mm, symbol Connector_Generic:Conn_01x01
- added J3: 5V, TestPoint:TestPoint_THTPad_2.5x2.5mm_Drill1.2mm, symbol Connector_Generic:Conn_01x01
- added J4: GND, TestPoint:TestPoint_THTPad_2.5x2.5mm_Drill1.2mm, symbol Connector_Generic:Conn_01x01
- added J9: V_Out, TestPoint:TestPoint_THTPad_4.0x4.0mm_Drill2.0mm, symbol Connector_Generic:Conn_01x01
- added U2: SY317, Package_TO_SOT_THT:TO-220-3_Vertical, symbol Regulator_Linear:L7805
- C10: renamed from C110; footprint (none) -> Capacitor_SMD:C_0603_1608Metric
- C11: renamed from C103; footprint (none) -> Capacitor_SMD:C_1210_3225Metric
- C12: renamed from C104; footprint (none) -> Capacitor_SMD:C_1210_3225Metric
- C13: renamed from C105; footprint (none) -> Capacitor_SMD:C_1210_3225Metric
- C14: renamed from C106; footprint (none) -> Capacitor_SMD:C_1210_3225Metric
- C15: renamed from C107; footprint (none) -> Capacitor_SMD:C_1210_3225Metric
- C2: renamed from C102; footprint (none) -> Capacitor_SMD:C_0603_1608Metric
- C3: renamed from C115; value 125n -> 100n; footprint (none) -> Capacitor_SMD:C_0603_1608Metric
- C4: renamed from C113; footprint (none) -> Capacitor_SMD:C_0603_1608Metric
- C5: renamed from C112; footprint (none) -> Capacitor_SMD:C_0603_1608Metric
- C6: renamed from C108; footprint (none) -> Capacitor_SMD:C_0603_1608Metric
- C7: renamed from C114; footprint (none) -> Capacitor_SMD:C_0603_1608Metric
- C8: renamed from C111; footprint (none) -> Capacitor_SMD:C_0603_1608Metric
- C9: renamed from C109; footprint (none) -> Capacitor_SMD:C_0603_1608Metric
- H1: renamed from H102; footprint (none) -> MountingHole:MountingHole_3.2mm_M3_DIN965
- H2: renamed from H101; footprint (none) -> MountingHole:MountingHole_3.2mm_M3_DIN965
- J1: renamed from J101; footprint (none) -> TestPoint:TestPoint_THTPad_4.0x4.0mm_Drill2.0mm
- J2: renamed from J102; footprint (none) -> TestPoint:TestPoint_THTPad_4.0x4.0mm_Drill2.0mm
- J5: renamed from J105; footprint (none) -> Connector_PinHeader_2.54mm:PinHeader_1x04_P2.54mm_Vertical
- J6: renamed from J106; footprint (none) -> Connector_PinHeader_2.54mm:PinHeader_1x04_P2.54mm_Vertical
- J7: renamed from J103; footprint (none) -> Connector_PinHeader_2.54mm:PinHeader_1x04_P2.54mm_Vertical
- J8: renamed from J104; footprint (none) -> Connector_PinHeader_2.54mm:PinHeader_1x04_P2.54mm_Vertical
- JP1: renamed from JP101; footprint (none) -> Jumper:SolderJumper-2_P1.3mm_Open_TrianglePad1.0x1.5mm
- JP2: renamed from JP102; footprint (none) -> Jumper:SolderJumper-2_P1.3mm_Open_TrianglePad1.0x1.5mm
- JP3: renamed from JP103; footprint (none) -> Jumper:SolderJumper-2_P1.3mm_Open_TrianglePad1.0x1.5mm
- JP4: renamed from JP104; footprint (none) -> Jumper:SolderJumper-2_P1.3mm_Open_TrianglePad1.0x1.5mm
- L1: renamed from L101; value SRP1038AA-2R2M -> SRP1038AA-2R2M; footprint (none) -> Inductor_SMD:L_Bourns_SRP1038C_10.0x10.0mm
- R1: renamed from R115; footprint (none) -> Resistor_SMD:R_0603_1608Metric
- R10: renamed from R109; footprint (none) -> Resistor_SMD:R_0603_1608Metric
- R11: renamed from R104; footprint (none) -> Resistor_SMD:R_0603_1608Metric
- R12: renamed from R105; footprint (none) -> Resistor_SMD:R_0603_1608Metric
- R13: renamed from R107; footprint (none) -> Resistor_SMD:R_0603_1608Metric
- R14: renamed from R102; footprint (none) -> Resistor_SMD:R_0603_1608Metric
- R15: renamed from R103; footprint (none) -> Resistor_SMD:R_0603_1608Metric
- R16: renamed from R106; footprint (none) -> Resistor_SMD:R_0603_1608Metric
- R17: renamed from R108; footprint (none) -> Resistor_SMD:R_0603_1608Metric
- R2: renamed from R116; footprint (none) -> Resistor_SMD:R_0603_1608Metric
- R3: renamed from R117; footprint (none) -> Resistor_SMD:R_0603_1608Metric
- R4: renamed from R113; footprint (none) -> Resistor_SMD:R_0603_1608Metric
- R5: renamed from R112; footprint (none) -> Resistor_SMD:R_0603_1608Metric
- R6: renamed from R114; footprint (none) -> Resistor_SMD:R_0603_1608Metric
- R7: renamed from R111; footprint (none) -> Resistor_SMD:R_0603_1608Metric
- R8: renamed from R110; footprint (none) -> Resistor_SMD:R_0603_1608Metric
- R9: renamed from R101; footprint (none) -> Resistor_SMD:R_0603_1608Metric
- U1: renamed from U101; footprint SIC471ED-T1-GE3:VREG_SIC471ED-T1-GE3 -> Eigene:VREG_SIC471ED-T1-GE3
Connections:
- net +24V: now also C1.1, U2.1 (IN)
- net +VDC: now also J9.1 (Pin_1)
- net GND: now also C1.2, J10.1 (Pin_1), J4.1 (Pin_1), U2.2 (GND)
- new net +5V: J3.1 (Pin_1), U2.3 (OUT)
Other:
- moved on the sheet: C2, J1, J2

Commit message: Overhaul
Other:
- note added: "Resistor Values for given Output Voltage: 5V: 52k5 6V: 65k 7V: 77k5 8V: 90k 9V: 102k5 10V: 115k 11V: 127k5 12V: 140k 13V: 152k5 14V: 165k 15V: 177k5 16V: 190k 17V: 202k5 18V: 215k"
- note removed: "CL32A476KOJNNNE"
- moved on the sheet: J3, J4, U2
