File: SY317/SY317.kicad_sch (KiCad schematic)
At the start: 14 parts, among them J1 Conn_01x03, U104 TPS56339DDC

Commit message: Overhaul
Parts:
- J1: value Conn_01x03 -> Pins
- R107: now not fitted
Other:
- note added: "UVLO Optional"
- moved on the sheet: C106, C107, C108, C109, C110, C111, J1, L101, R108, R109, R110, RV1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
